File: vrb.kicad_pcb (KiCad board)
At the start: 2 copper layers, 73 x 69 mm, 174 parts, among them J1 SM04B-GHS, J10 MiniFit, J11 XT30, J2 SM04B-GHS, J3 MiniFit, J4 MiniFit, J5 Pixhawk 1, J6 Pixhawk 2, J7 SM04B-GHS, J8 DEBUG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

Commit message: work on layout
Parts:
- moved C54 1.00 mm to (134.3, 114.8)
- moved C55 1.00 mm to (136.8, 117.7)
- moved C57 1.00 mm to (138.6, 116.3)
- moved R71 1.00 mm to (139.8, 116.3)
- moved R72 1.00 mm to (139.2, 114.6)
- moved Y1 1.00 mm to (136.4, 115.4)
- moved C38 0.78 mm to (134.6, 112.4)
- moved C39 0.78 mm to (133.5, 112.4)
Routing:
- net GND: track 57.1 -> 60.2 mm, vias 75 -> 78
- net /XIN: track 5.17 -> 7.30 mm
- net Net-(U1-VBAT): track 2.78 -> 4.81 mm, vias 1 -> 3
- net /XOUT: track 7.22 -> 9.22 mm
- net /nRST: track 6.31 -> 8.31 mm
Other:
- board size 73 x 69 mm -> 75 x 69 mm
