File: passthrough.kicad_sch (KiCad schematic)
At the start: 14 parts, among them J10 MiniFit, J5 Pixhawk 1, J6 Pixhawk 2, U17 TA2528

Commit message: move to 6 layer
Parts:
- U17: value TA2528 -> TLA2528
Changed lines of the file:
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@@
 			)
 		)
-		(property "Value" "TA2528"
+		(property "Value" "TLA2528"
 			(at 205.3433 74.93 0)
 			(effects
