File: vrb.kicad_sch (KiCad schematic)
At the start: 9 parts, among them J11 XT30, J12 Mezzanine, U1 STM32G0B1CBUx

Commit message: finish layout
Parts:
- added D20: RED, LED_SMD:LED_0603_1608Metric, symbol Device:LED
- added R78: 330, Resistor_SMD:R_0402_1005Metric, symbol Device:R
Connections:
- net GND: now also R78.2
- net +3V3: now reaches C38.1, C39.1, U1.4 (VBAT), U1.6 (VDD)
- net FAULT: now reaches U1.29 (PA9/UCPD1_DBCC1)
- net FAULT: now also D20.2 (A)
- new net: D20.1 (K), R78.1
- no-connect marks 4 -> 3
Other:
- note added: "Fault LED"
- note removed: "TODO: Input power mux?"
- moved on the sheet: C38, C39, U1

Commit message: optimize components, update schematic pdf
Parts:
- H1, H2, H3, H4: footprint MountingHole:MountingHole_3.2mm_M3_Pad_TopBottom -> MountingHole:MountingHole_3.2mm_M3_Pad_Via
Changed lines of the file:
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@@
 			)
 		)
-		(property "Footprint" "MountingHole:MountingHole_3.2mm_M3_Pad_TopBottom"
+		(property "Footprint" "MountingHole:MountingHole_3.2mm_M3_Pad_Via"
 			(at 210.82 133.35 0)
 			(effects
@@
 			)
 		)
-		(property "Footprint" "MountingHole:MountingHole_3.2mm_M3_Pad_TopBottom"
+		(property "Footprint" "MountingHole:MountingHole_3.2mm_M3_Pad_Via"
 			(at 195.58 133.35 0)
 			(effects
@@
 			)
 		)
-		(property "Footprint" "MountingHole:MountingHole_3.2mm_M3_Pad_TopBottom"
+		(property "Footprint" "MountingHole:MountingHole_3.2mm_M3_Pad_Via"
 			(at 200.66 133.35 0)
 			(effects
@@
 			)
 		)
-		(property "Footprint" "MountingHole:MountingHole_3.2mm_M3_Pad_TopBottom"
+		(property "Footprint" "MountingHole:MountingHole_3.2mm_M3_Pad_Via"
 			(at 205.74 133.35 0)
 			(effects
