File: vrb.kicad_sch (KiCad schematic)
At the start: 13 parts, among them J11 XT30, J12 Mezzanine, J14 Conn_01x02, U1 STM32G0B1CBUx

Commit message: improvements with derick
Parts:
- removed D20: RED, LED_SMD:LED_0603_1608Metric, symbol Device:LED
- removed R78: 330, Resistor_SMD:R_0402_1005Metric, symbol Device:R
- added TP12: GND, TestPoint:TestPoint_Loop_D2.50mm_Drill1.0mm, symbol Connector:TestPoint
- J14: now left out of the parts list
Connections:
- net GND: now also TP12.1
- net FAULT renamed nFAULT
Other:
- sheet Passthrough Ports ports: added ~{FAULT}; removed none
- note removed: "Fault LED"
- note removed: "TODO: Make this fault LED powered by VBAT"
- moved on the sheet: J11

Commit message: final export of r1 after changes
Connections:
- net IPAYLOAD renamed IPAYLOAD1
- net RESV0 renamed IPAYLOAD2
- net RESV1 renamed IPAYLOAD3
- net RESV2 renamed VBAT_SCALED
Other:
- sheet Passthrough Ports ports: added IPAYLOAD1, IPAYLOAD2, IPAYLOAD3, VBAT_SCALED; removed IPAYLOAD, RESV0, RESV1, RESV2
Changed lines of the file:
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@@
 	(wire
 		(pts
+			(xy 256.54 119.38) (xy 270.51 119.38)
+		)
+		(stroke
+			(width 0)
+			(type default)
+		)
+	)
+	(wire
+		(pts
 			(xy 21.59 83.82) (xy 38.1 83.82)
 		)
@@
 	(wire
 		(pts
+			(xy 256.54 114.3) (xy 270.51 114.3)
+		)
+		(stroke
+			(width 0)
+			(type default)
+		)
+	)
+	(wire
+		(pts
 			(xy 144.78 182.88) (xy 151.13 182.88)
 		)
@@
 	(wire
 		(pts
+			(xy 256.54 106.68) (xy 270.51 106.68)
+		)
+		(stroke
+			(width 0)
+			(type default)
+		)
+	)
+	(wire
+		(pts
 			(xy 243.84 83.82) (xy 241.3 83.82)
 		)
@@
 	(wire
 		(pts
+			(xy 256.54 104.14) (xy 270.51 104.14)
+		)
+		(stroke
+			(width 0)
+			(type default)
+		)
+	)
+	(wire
+		(pts
 			(xy 129.54 31.75) (xy 146.05 31.75)
 		)
@@
 	(wire
 		(pts
-			(xy 256.54 106.68) (xy 267.97 106.68)
-		)
-		(stroke
-			(width 0)
-			(type default)
-		)
-	)
-	(wire
-		(pts
 			(xy 76.2 173.99) (xy 95.25 173.99)
 		)
@@
 	(wire
 		(pts
-			(xy 256.54 119.38) (xy 267.97 119.38)
-		)
-		(stroke
-			(width 0)
-			(type default)
-		)
-	)
-	(wire
-		(pts
-			(xy 256.54 116.84) (xy 267.97 116.84)
+			(xy 256.54 109.22) (xy 270.51 109.22)
 		)
 		(stroke
@@
 	(wire
 		(pts
-			(xy 256.54 109.22) (xy 267.97 109.22)
-		)
-		(stroke
-			(width 0)
-			(type default)
-		)
-	)
-	(wire
-		(pts
 			(xy 93.98 99.06) (xy 114.3 99.06)
 		)
@@
 	(wire
 		(pts
-			(xy 256.54 104.14) (xy 267.97 104.14)
-		)
-		(stroke
-			(width 0)
-			(type default)
-		)
-	)
-	(wire
-		(pts
 			(xy 205.74 137.16) (xy 210.82 137.16)
 		)
@@
 	(wire
 		(pts
-			(xy 256.54 114.3) (xy 267.97 114.3)
-		)
-		(stroke
-			(width 0)
-			(type default)
-		)
-	)
-	(wire
-		(pts
 			(xy 241.3 91.44) (xy 243.84 91.44)
 		)
@@
 	(wire
 		(pts
-			(xy 179.07 34.29) (xy 194.31 34.29)
+			(xy 256.54 116.84) (xy 270.51 116.84)
 		)
 		(stroke
@@
 	(wire
 		(pts
-			(xy 259.08 71.12) (xy 259.08 73.66)
+			(xy 179.07 34.29) (xy 194.31 34.29)
 		)
 		(stroke
@@
 	(wire
 		(pts
-			(xy 259.08 78.74) (xy 259.08 81.28)
+			(xy 259.08 71.12) (xy 259.08 73.66)
 		)
 		(stroke
@@
 	(wire
 		(pts
-			(xy 179.07 27.94) (xy 194.31 27.94)
+			(xy 259.08 78.74) (xy 259.08 81.28)
 		)
 		(stroke
@@
 	(wire
 		(pts
-			(xy 93.98 83.82) (xy 114.3 83.82)
+			(xy 179.07 27.94) (xy 194.31 27.94)
 		)
 		(stroke
@@
 	(wire
 		(pts
-			(xy 256.54 111.76) (xy 267.97 111.76)
+			(xy 93.98 83.82) (xy 114.3 83.82)
 		)
 		(stroke
@@
 	(wire
 		(pts
+			(xy 256.54 101.6) (xy 270.51 101.6)
+		)
+		(stroke
+			(width 0)
+			(type default)
+		)
+	)
+	(wire
+		(pts
 			(xy 129.54 86.36) (xy 146.05 86.36)
 		)
@@
 	(wire
 		(pts
-			(xy 256.54 101.6) (xy 267.97 101.6)
+			(xy 241.3 38.1) (xy 241.3 35.56)
 		)
 		(stroke
@@
 	(wire
 		(pts
-			(xy 241.3 38.1) (xy 241.3 35.56)
+			(xy 21.59 50.8) (xy 38.1 50.8)
 		)
 		(stroke
@@
 	(wire
 		(pts
-			(xy 21.59 50.8) (xy 38.1 50.8)
+			(xy 256.54 111.76) (xy 270.51 111.76)
 		)
 		(stroke
@@
 		)
 	)
-	(label "RESV1"
-		(at 267.97 116.84 180)
+	(label "IPAYLOAD3"
+		(at 270.51 116.84 180)
 		(effects
 			(font
@@
 	)
 	(label "IESC2"
-		(at 267.97 104.14 180)
+		(at 270.51 104.14 180)
 		(effects
 			(font
@@
 		)
 	)
-	(label "RESV2"
+	(label "VBAT_SCALED"
 		(at 76.2 191.77 0)
 		(effects
@@
 		)
 	)
-	(label "RESV2"
-		(at 267.97 119.38 180)
+	(label "VBAT_SCALED"
+		(at 270.51 119.38 180)
 		(effects
 			(font
@@
 	)
 	(label "IESC1"
-		(at 267.97 101.6 180)
+		(at 270.51 101.6 180)
 		(effects
 			(font
@@
 	)
 	(label "IESC3"
-		(at 267.97 106.68 180)
+		(at 270.51 106.68 180)
 		(effects
 			(font
@@
 		)
 	)
-	(label "IPAYLOAD"
+	(label "IPAYLOAD1"
 		(at 76.2 184.15 0)
 		(effects
@@
 	)
 	(label "IESC4"
-		(at 267.97 109.22 180)
+		(at 270.51 109.22 180)
 		(effects
 			(font
@@
 		)
 	)
-	(label "IPAYLOAD"
-		(at 267.97 111.76 180)
+	(label "IPAYLOAD1"
+		(at 270.51 111.76 180)
 		(effects
 			(font
@@
 		)
 	)
-	(label "RESV0"
-		(at 267.97 114.3 180)
+	(label "IPAYLOAD2"
+		(at 270.51 114.3 180)
 		(effects
 			(font
@@
 		)
 	)
-	(label "RESV0"
+	(label "IPAYLOAD2"
 		(at 76.2 186.69 0)
 		(effects
@@
 		)
 	)
-	(label "RESV1"
+	(label "IPAYLOAD3"
 		(at 76.2 189.23 0)
 		(effects
@@
 			)
 		)
-		(pin "IPAYLOAD" input
+		(pin "IPAYLOAD1" input
 			(at 95.25 184.15 180)
 			(effects
@@
 			)
 		)
-		(pin "RESV0" input
+		(pin "IPAYLOAD2" input
 			(at 95.25 186.69 180)
 			(effects
@@
 			)
 		)
-		(pin "RESV1" input
+		(pin "IPAYLOAD3" input
 			(at 95.25 189.23 180)
 			(effects
@@
 			)
 		)
-		(pin "RESV2" input
+		(pin "VBAT_SCALED" input
 			(at 95.25 191.77 180)
 			(effects

Commit message: updated layout for fault led with new circuit, rerouted
Parts:
- renumbered C38 to C1, C39 to C2, J11 to J1, J12 to J2, J14 to J3, R79 to R1, TP12 to TP1
Changed lines of the file:
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@@
 		(on_board yes)
 		(dnp no)
-		(property "Reference" "#PWR0154"
+		(property "Reference" "#PWR011"
 			(at 241.3 128.27 0)
 			(effects
@@
 			(project ""
 				(path "/59a9b615-ea12-4a8c-9228-b32f861e8d75"
-					(reference "#PWR0154")
+					(reference "#PWR011")
 					(unit 1)
 				)
@@
 		(dnp no)
 		(fields_autoplaced yes)
-		(property "Reference" "J11"
+		(property "Reference" "J1"
 			(at 251.46 33.0199 0)
 			(effects
@@
 			(project ""
 				(path "/59a9b615-ea12-4a8c-9228-b32f861e8d75"
-					(reference "J11")
+					(reference "J1")
 					(unit 1)
 				)
@@
 		(dnp no)
 		(fields_autoplaced yes)
-		(property "Reference" "#PWR01"
+		(property "Reference" "#PWR012"
 			(at 66.04 143.51 0)
 			(effects
@@
 			(project ""
 				(path "/59a9b615-ea12-4a8c-9228-b32f861e8d75"
-					(reference "#PWR01")
+					(reference "#PWR012")
 					(unit 1)
 				)
@@
 		(dnp no)
 		(fields_autoplaced yes)
-		(property "Reference" "#PWR0136"
+		(property "Reference" "#PWR010"
 			(at 191.77 104.14 0)
 			(effects
@@
 			(project "vrb"
 				(path "/59a9b615-ea12-4a8c-9228-b32f861e8d75"
-					(reference "#PWR0136")
+					(reference "#PWR010")
 					(unit 1)
 				)
@@
 		(dnp no)
 		(fields_autoplaced yes)
-		(property "Reference" "C39"
+		(property "Reference" "C2"
 			(at 87.63 30.4862 0)
 			(effects
@@
 			(project "vrb"
 				(path "/59a9b615-ea12-4a8c-9228-b32f861e8d75"
-					(reference "C39")
+					(reference "C2")
 					(unit 1)
 				)
@@
 		(dnp no)
 		(fields_autoplaced yes)
-		(property "Reference" "#PWR0126"
+		(property "Reference" "#PWR03"
 			(at 260.35 36.83 0)
 			(effects
@@
 			(project "vrb"
 				(path "/59a9b615-ea12-4a8c-9228-b32f861e8d75"
-					(reference "#PWR0126")
+					(reference "#PWR03")
 					(unit 1)
 				)
@@
 		(dnp no)
 		(fields_autoplaced yes)
-		(property "Reference" "J12"
+		(property "Reference" "J2"
 			(at 250.19 64.77 0)
 			(effects
@@
 			(project ""
 				(path "/59a9b615-ea12-4a8c-9228-b32f861e8d75"
-					(reference "J12")
+					(reference "J2")
 					(unit 1)
 				)
@@
 		(dnp no)
 		(fields_autoplaced yes)
-		(property "Reference" "#PWR0127"
+		(property "Reference" "#PWR04"
 			(at 269.24 41.91 0)
 			(effects
@@
 			(project "vrb"
 				(path "/59a9b615-ea12-4a8c-9228-b32f861e8d75"
-					(reference "#PWR0127")
+					(reference "#PWR04")
 					(unit 1)
 				)
@@
 		(dnp no)
 		(fields_autoplaced yes)
-		(property "Reference" "#PWR0189"
+		(property "Reference" "#PWR06"
 			(at 227.33 43.18 0)
 			(effects
@@
 			(project "vrb"
 				(path "/59a9b615-ea12-4a8c-9228-b32f861e8d75"
-					(reference "#PWR0189")
+					(reference "#PWR06")
 					(unit 1)
 				)
@@
 		(on_board yes)
 		(dnp no)
-		(property "Reference" "#PWR0116"
+		(property "Reference" "#PWR05"
 			(at 85.09 43.18 0)
 			(effects
@@
 			(project ""
 				(path "/59a9b615-ea12-4a8c-9228-b32f861e8d75"
-					(reference "#PWR0116")
+					(reference "#PWR05")
 					(unit 1)
 				)
@@
 		(dnp no)
 		(fields_autoplaced yes)
-		(property "Reference" "#PWR0130"
+		(property "Reference" "#PWR08"
 			(at 191.77 72.39 0)
 			(effects
@@
 			(project ""
 				(path "/59a9b615-ea12-4a8c-9228-b32f861e8d75"
-					(reference "#PWR0130")
+					(reference "#PWR08")
 					(unit 1)
 				)
@@
 		(dnp no)
 		(fields_autoplaced yes)
-		(property "Reference" "#PWR0180"
+		(property "Reference" "#PWR014"
 			(at 144.78 173.99 0)
 			(effects
@@
 			(project ""
 				(path "/59a9b615-ea12-4a8c-9228-b32f861e8d75"
-					(reference "#PWR0180")
+					(reference "#PWR014")
 					(unit 1)
 				)
@@
 		(dnp no)
 		(fields_autoplaced yes)
-		(property "Reference" "C38"
+		(property "Reference" "C1"
 			(at 77.47 30.4862 0)
 			(effects
@@
 			(project ""
 				(path "/59a9b615-ea12-4a8c-9228-b32f861e8d75"
-					(reference "C38")
+					(reference "C1")
 					(unit 1)
 				)
@@
 		(on_board yes)
 		(dnp no)
-		(property "Reference" "#PWR0165"
+		(property "Reference" "#PWR01"
 			(at 66.04 29.21 0)
 			(effects
@@
 			(project ""
 				(path "/59a9b615-ea12-4a8c-9228-b32f861e8d75"
-					(reference "#PWR0165")
+					(reference "#PWR01")
 					(unit 1)
 				)
@@
 		(dnp no)
 		(fields_autoplaced yes)
-		(property "Reference" "#PWR0181"
+		(property "Reference" "#PWR015"
 			(at 148.59 194.31 0)
 			(effects
@@
 			(project ""
 				(path "/59a9b615-ea12-4a8c-9228-b32f861e8d75"
-					(reference "#PWR0181")
+					(reference "#PWR015")
 					(unit 1)
 				)
@@
 		(dnp no)
 		(fields_autoplaced yes)
-		(property "Reference" "#PWR0152"
+		(property "Reference" "#PWR09"
 			(at 259.08 72.39 0)
 			(effects
@@
 			(project "vrb"
 				(path "/59a9b615-ea12-4a8c-9228-b32f861e8d75"
-					(reference "#PWR0152")
+					(reference "#PWR09")
 					(unit 1)
 				)
@@
 		(dnp no)
 		(fields_autoplaced yes)
-		(property "Reference" "#PWR0125"
+		(property "Reference" "#PWR07"
 			(at 241.3 44.45 0)
 			(effects
@@
 			(project ""
 				(path "/59a9b615-ea12-4a8c-9228-b32f861e8d75"
-					(reference "#PWR0125")
+					(reference "#PWR07")
 					(unit 1)
 				)
@@
 		(dnp no)
 		(fields_autoplaced yes)
-		(property "Reference" "R79"
+		(property "Reference" "R1"
 			(at 147.32 175.2599 0)
 			(effects
@@
 			(project ""
 				(path "/59a9b615-ea12-4a8c-9228-b32f861e8d75"
-					(reference "R79")
+					(reference "R1")
 					(unit 1)
 				)
@@
 		(dnp no)
 		(fields_autoplaced yes)
-		(property "Reference" "#FLG01"
+		(property "Reference" "#FLG02"
 			(at 260.35 37.465 0)
 			(effects
@@
 			(project ""
 				(path "/59a9b615-ea12-4a8c-9228-b32f861e8d75"
-					(reference "#FLG01")
+					(reference "#FLG02")
 					(unit 1)
 				)
@@
 		(dnp no)
 		(fields_autoplaced yes)
-		(property "Reference" "#PWR0124"
+		(property "Reference" "#PWR02"
 			(at 241.3 34.29 0)
 			(effects
@@
 			(project ""
 				(path "/59a9b615-ea12-4a8c-9228-b32f861e8d75"
-					(reference "#PWR0124")
+					(reference "#PWR02")
 					(unit 1)
 				)
@@
 		(dnp no)
 		(fields_autoplaced yes)
-		(property "Reference" "TP12"
+		(property "Reference" "TP1"
 			(at 229.87 29.7179 0)
 			(effects
@@
 			(project ""
 				(path "/59a9b615-ea12-4a8c-9228-b32f861e8d75"
-					(reference "TP12")
+					(reference "TP1")
 					(unit 1)
 				)
@@
 		(dnp no)
 		(fields_autoplaced yes)
-		(property "Reference" "#FLG02"
+		(property "Reference" "#FLG01"
 			(at 269.24 31.115 0)
 			(effects
@@
 			(project "vrb"
 				(path "/59a9b615-ea12-4a8c-9228-b32f861e8d75"
-					(reference "#FLG02")
+					(reference "#FLG01")
 					(unit 1)
 				)
@@
 		(dnp no)
 		(fields_autoplaced yes)
-		(property "Reference" "J14"
+		(property "Reference" "J3"
 			(at 158.75 182.8799 0)
 			(effects
@@
 			(project ""
 				(path "/59a9b615-ea12-4a8c-9228-b32f861e8d75"
-					(reference "J14")
+					(reference "J3")
 					(unit 1)
 				)
@@
 		(dnp no)
 		(fields_autoplaced yes)
-		(property "Reference" "#PWR078"
+		(property "Reference" "#PWR013"
 			(at 195.58 144.78 0)
 			(effects
@@
 			(project ""
 				(path "/59a9b615-ea12-4a8c-9228-b32f861e8d75"
-					(reference "#PWR078")
-					(unit 1)
-				)
+					(reference "#PWR013")
+					(unit 1)
+				)
