File: port.kicad_sch (KiCad schematic)
At the start: 16 parts, among them J4 MiniFit, U15 TPS2121

Commit message: improvements with derick
Parts:
- TP7: now left out of the parts list
Changed lines of the file:
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@@
 		(unit 1)
 		(exclude_from_sim no)
-		(in_bom yes)
+		(in_bom no)
 		(on_board yes)
 		(dnp no)

Commit message: updated layout for fault led with new circuit, rerouted
Parts:
- renumbered C33 to C37, C34 to C38, C36 to C39, C35 to C40, D13 to D14, J4 to J8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
