File: rcc.kicad_sch (KiCad schematic)
At the start: 7 parts, among them J8 DEBUG, Y1 XRCGB16M000FXN20R0

Commit message: improvements with derick
Parts:
- J8: now left out of the parts list
Changed lines of the file:
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@@
 		(unit 1)
 		(exclude_from_sim no)
-		(in_bom yes)
+		(in_bom no)
 		(on_board yes)
 		(dnp no)

Commit message: updated layout for fault led with new circuit, rerouted
Parts:
- renumbered C54 to C48, C55 to C49, C57 to C50, J8 to J14, R71 to R83, R72 to R84
Changed lines of the file:
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@@
 		(dnp no)
 		(fields_autoplaced yes)
-		(property "Reference" "R71"
+		(property "Reference" "R83"
 			(at 43.18 39.3699 0)
 			(effects
@@
 			(project "vrb"
 				(path "/59a9b615-ea12-4a8c-9228-b32f861e8d75/0d4bd9cc-8b27-4bd8-8a00-67e0b9520a22"
-					(reference "R71")
+					(reference "R83")
 					(unit 1)
 				)
@@
 		(dnp no)
 		(fields_autoplaced yes)
-		(property "Reference" "#PWR0140"
+		(property "Reference" "#PWR0171"
 			(at 29.21 66.04 0)
 			(effects
@@
 			(project "vrb"
 				(path "/59a9b615-ea12-4a8c-9228-b32f861e8d75/0d4bd9cc-8b27-4bd8-8a00-67e0b9520a22"
-					(reference "#PWR0140")
+					(reference "#PWR0171")
 					(unit 1)
 				)
@@
 		(dnp no)
 		(fields_autoplaced yes)
-		(property "Reference" "#PWR0141"
+		(property "Reference" "#PWR0172"
 			(at 40.64 66.04 0)
 			(effects
@@
 			(project "vrb"
 				(path "/59a9b615-ea12-4a8c-9228-b32f861e8d75/0d4bd9cc-8b27-4bd8-8a00-67e0b9520a22"
-					(reference "#PWR0141")
+					(reference "#PWR0172")
 					(unit 1)
 				)
@@
 		(dnp no)
 		(fields_autoplaced yes)
-		(property "Reference" "C55"
+		(property "Reference" "C49"
 			(at 166.37 50.165 0)
 			(effects
@@
 			(project "vrb"
 				(path "/59a9b615-ea12-4a8c-9228-b32f861e8d75/0d4bd9cc-8b27-4bd8-8a00-67e0b9520a22"
-					(reference "C55")
+					(reference "C49")
 					(unit 1)
 				)
@@
 		(dnp no)
 		(fields_autoplaced yes)
-		(property "Reference" "#PWR0135"
+		(property "Reference" "#PWR0170"
 			(at 162.56 63.5 0)
 			(effects
@@
 			(project "vrb"
 				(path "/59a9b615-ea12-4a8c-9228-b32f861e8d75/0d4bd9cc-8b27-4bd8-8a00-67e0b9520a22"
-					(reference "#PWR0135")
+					(reference "#PWR0170")
 					(unit 1)
 				)
@@
 		(dnp no)
 		(fields_autoplaced yes)
-		(property "Reference" "#PWR079"
+		(property "Reference" "#PWR0166"
 			(at 104.14 41.91 0)
 			(effects
@@
 			(project "vrb"
 				(path "/59a9b615-ea12-4a8c-9228-b32f861e8d75/0d4bd9cc-8b27-4bd8-8a00-67e0b9520a22"
-					(reference "#PWR079")
+					(reference "#PWR0166")
 					(unit 1)
 				)
@@
 		(on_board yes)
 		(dnp no)
-		(property "Reference" "C54"
+		(property "Reference" "C48"
 			(at 142.24 49.53 0)
 			(effects
@@
 			(project "vrb"
 				(path "/59a9b615-ea12-4a8c-9228-b32f861e8d75/0d4bd9cc-8b27-4bd8-8a00-67e0b9520a22"
-					(reference "C54")
+					(reference "C48")
 					(unit 1)
 				)
@@
 		(dnp no)
 		(fields_autoplaced yes)
-		(property "Reference" "#PWR0133"
+		(property "Reference" "#PWR0167"
 			(at 156.21 58.42 0)
 			(effects
@@
 			(project "vrb"
 				(path "/59a9b615-ea12-4a8c-9228-b32f861e8d75/0d4bd9cc-8b27-4bd8-8a00-67e0b9520a22"
-					(reference "#PWR0133")
+					(reference "#PWR0167")
 					(unit 1)
 				)
@@
 		(dnp no)
 		(fields_autoplaced yes)
-		(property "Reference" "#PWR0134"
+		(property "Reference" "#PWR0169"
 			(at 149.86 63.5 0)
 			(effects
@@
 			(project "vrb"
 				(path "/59a9b615-ea12-4a8c-9228-b32f861e8d75/0d4bd9cc-8b27-4bd8-8a00-67e0b9520a22"
-					(reference "#PWR0134")
+					(reference "#PWR0169")
 					(unit 1)
 				)
@@
 		(on_board yes)
 		(dnp yes)
-		(property "Reference" "R72"
+		(property "Reference" "R84"
 			(at 31.75 50.8 0)
 			(effects
@@
 			(project "vrb"
 				(path "/59a9b615-ea12-4a8c-9228-b32f861e8d75/0d4bd9cc-8b27-4bd8-8a00-67e0b9520a22"
-					(reference "R72")
+					(reference "R84")
 					(unit 1)
 				)
@@
 		(dnp no)
 		(fields_autoplaced yes)
-		(property "Reference" "J8"
+		(property "Reference" "J14"
 			(at 114.3 44.4499 0)
 			(effects
@@
 			(project "vrb"
 				(path "/59a9b615-ea12-4a8c-9228-b32f861e8d75/0d4bd9cc-8b27-4bd8-8a00-67e0b9520a22"
-					(reference "J8")
+					(reference "J14")
 					(unit 1)
 				)
@@
 		(dnp no)
 		(fields_autoplaced yes)
-		(property "Reference" "#PWR0138"
+		(property "Reference" "#PWR0164"
 			(at 40.64 38.1 0)
 			(effects
@@
 			(project "vrb"
 				(path "/59a9b615-ea12-4a8c-9228-b32f861e8d75/0d4bd9cc-8b27-4bd8-8a00-67e0b9520a22"
-					(reference "#PWR0138")
+					(reference "#PWR0164")
 					(unit 1)
 				)
@@
 		(dnp no)
 		(fields_autoplaced yes)
-		(property "Reference" "#PWR0117"
+		(property "Reference" "#PWR0168"
 			(at 104.14 59.69 0)
 			(effects
@@
 			(project "vrb"
 				(path "/59a9b615-ea12-4a8c-9228-b32f861e8d75/0d4bd9cc-8b27-4bd8-8a00-67e0b9520a22"
-					(reference "#PWR0117")
+					(reference "#PWR0168")
 					(unit 1)
 				)
@@
 		(dnp no)
 		(fields_autoplaced yes)
-		(property "Reference" "#PWR0131"
+		(property "Reference" "#PWR0165"
 			(at 151.13 43.18 0)
 			(effects
@@
 			(project "vrb"
 				(path "/59a9b615-ea12-4a8c-9228-b32f861e8d75/0d4bd9cc-8b27-4bd8-8a00-67e0b9520a22"
-					(reference "#PWR0131")
+					(reference "#PWR0165")
 					(unit 1)
 				)
@@
 		(dnp no)
 		(fields_autoplaced yes)
-		(property "Reference" "C57"
+		(property "Reference" "C50"
 			(at 44.45 52.07 0)
 			(effects
@@
 			(project "vrb"
 				(path "/59a9b615-ea12-4a8c-9228-b32f861e8d75/0d4bd9cc-8b27-4bd8-8a00-67e0b9520a22"
-					(reference "C57")
-					(unit 1)
-				)
+					(reference "C50")
+					(unit 1)
+				)
