File: regulator.kicad_sch (KiCad schematic)
At the start: 20 parts, among them U3 LMR51635, U4 INA180A2

Commit message: improvements with derick
Parts:
- D4: value BLUE -> GREEN
- TP1: now left out of the parts list
Other:
- note added: "fSW = 400KHz, VOUT = 5.2V, IOUT = 3.5A L = 10uH, COUT = 2x 33uF [16V], RFBT = 56.1K ~ 56K For 5.0V, RFBT = 53.6K"
- note removed: "fSW = 400KHz, VOUT = 5.2V, IOUT = 3.5A L = 10uH, COUT = 2x 33uF [16V], RFBT = 56.1K For 5.0V, RFBT = 53.6K"
Changed lines of the file:
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@@
 		)
 	)
-	(text "fSW = 400KHz, VOUT = 5.2V, IOUT = 3.5A\nL = 10uH, COUT = 2x 33uF [16V], RFBT = 56.1K\nFor 5.0V, RFBT = 53.6K"
+	(text "fSW = 400KHz, VOUT = 5.2V, IOUT = 3.5A\nL = 10uH, COUT = 2x 33uF [16V], RFBT = 56.1K ~ 56K\nFor 5.0V, RFBT = 53.6K"
 		(exclude_from_sim no)
 		(at 30.48 29.21 0)
@@
 		(unit 1)
 		(exclude_from_sim no)
-		(in_bom yes)
+		(in_bom no)
 		(on_board yes)
 		(dnp no)
@@
 			)
 		)
-		(property "Value" "BLUE"
+		(property "Value" "GREEN"
 			(at 73.66 100.33 0)
 			(effects

Commit message: updated layout for fault led with new circuit, rerouted
Parts:
- renumbered C7 to C10, C8 to C11, C47 to C6, C4 to C7, C5 to C8, C6 to C9, D4 to D5, R9 to R10, R10 to R11, R11 to R12, R12 to R13, R13 to R14, R14 to R15, R7 to R8, R8 to R9, TP1 to TP3
