File: regulator_onboard.kicad_sch (KiCad schematic)
At the start: 12 parts, among them U16 TLV71333PDQN, U18 TPS2116DRL

Commit message: finish layout
Parts:
- U16: value TLV71333PDQN -> TLV71333PDBVR; symbol TLV71333PDQ:TLV71333PDQN -> TLV71333PDQ:TLV71333PDBVR
Connections:
- net +3V3: now also U16.5 (OUT); no longer U16.1 (OUT)
- net +5V: now also U16.1 (IN); no longer U16.4 (IN)
- net GND: no longer U16.5 (GND)
Other:
- moved on the sheet: C40, C41, D18, R70, U16

Commit message: improvements with derick
Parts:
- added TP10: TestPoint, TestPoint:TestPoint_Pad_1.0x1.0mm, symbol Connector:TestPoint
- TP9: now left out of the parts list
Connections:
- net +3V3: now also TP10.1
Other:
- moved on the sheet: C40, C41, D18, R70, U16

Commit message: updated layout for fault led with new circuit, rerouted
Parts:
- renumbered C43 to C51, C45 to C52, C40 to C53, C41 to C54, D18 to D21, R74 to R85, R70 to R86, R77 to R87, R76 to R88, TP10 to TP11, TP9 to TP12, U16 to U17
